File: AppleVGA/AppleVGA_Connections.kicad_sch (KiCad schematic)
At the start: 7 parts, among them J1 AppleIIBus, J2 VGA, J3 VGA, SW1 SW_Push

Commit message: Add files via upload
Parts:
- removed J2: VGA, Connector_PinHeader_2.54mm:PinHeader_1x08_P2.54mm_Vertical, symbol Connector_Generic:Conn_01x08
- removed J3: VGA, Connector_Dsub:DSUB-15-HD_Female_Horizontal_P2.29x1.98mm_EdgePinOffset3.03mm_Housed_MountingHolesOffset4.94mm, symbol Connector:DB15_Female_HighDensity_MountingHoles
- added J2: VGA, Connector_PinSocket_2.54mm:PinSocket_2x08_P2.54mm_Vertical, symbol Connector_Generic:Conn_02x08_Odd_Even
Connections:
- net GND: now also J2.10 (Pin_10), J2.16 (Pin_16), J2.5 (Pin_5), J2.6 (Pin_6), J2.7 (Pin_7), J2.8 (Pin_8)
- net VGA_B: now also J2.3 (Pin_3)
- net VGA_G: now also J2.2 (Pin_2)
- net VGA_HSYNC: now also J2.13 (Pin_13)
- net VGA_R: now also J2.1 (Pin_1)
- net VGA_VSYNC: now also J2.14 (Pin_14)
Other:
- moved on the sheet: C1, C3, C5, SW1
